Commit message: Fix errors

File: rover_description/urdf/rover.urdf.xacro (robot description, xacro)
@@ -56,5 +56,5 @@
                     <cylinder radius = "${wheel_radius}" length = "${wheel_length}" />
                 </geometry>
-                <origin xyz = "0 0 0" rpy = "0 0 0" />
+                <origin xyz = "0 0 0" rpy = "${pi / 2.0} 0 0" />
                 <material name = "gray" />
             </visual>
@@ -111,7 +111,7 @@
         <origin xyz = "0 0 ${wheel_radius}" rpy = "0 0 0" />
     </joint>
-    <xacro:wheel_joint prefix = "front_right" x = "{base_length / 4.0}" y = "${-(base_width + wheel_length) / 2.0}" />
-    <xacro:wheel_joint prefix = "front_left" x = "{base_length / 4.0}" y = "${(base_width + wheel_length) / 2.0}" />
-    <xacro:wheel_joint prefix = "back_right" x = "{-base_length / 4.0}" y = "${-(base_width + wheel_length) / 2.0}" />
-    <xacro:wheel_joint prefix = "back_left" x = "{-base_length / 4.0}" y = "${(base_width + wheel_length) / 2.0}" />
+    <xacro:wheel_joint prefix = "front_right" x = "${base_length / 4.0}" y = "${-(base_width + wheel_length) / 2.0}" />
+    <xacro:wheel_joint prefix = "front_left" x = "${base_length / 4.0}" y = "${(base_width + wheel_length) / 2.0}" />
+    <xacro:wheel_joint prefix = "back_right" x = "${-base_length / 4.0}" y = "${-(base_width + wheel_length) / 2.0}" />
+    <xacro:wheel_joint prefix = "back_left" x = "${-base_length / 4.0}" y = "${(base_width + wheel_length) / 2.0}" />
 </robot>

Commit message: Add JointStatePublisher plugin

File: rover_description/urdf/rover.urdf.xacro (robot description, xacro)
@@ -37,17 +37,4 @@
         </inertial>
     </xacro:macro>
-    <!-- May not be necessary ! -->
-    <!-- <xacro:macro name = "sphere_inertia" params = "m r o_xyz o_rpy">
-        <inertial>
-            <mass value = "${m}"/>
-            <origin xyz = "${o_xyz}" rpy = "${o_rpy}" />
-            <inertia
-                ixx = "${(2 / 5) * m * r * r}"
-                iyy = "${(2 / 5) * m * r * r}"
-                izz = "${(2 / 5) * m * r * r}"
-                ixy = "0" iyz = "0" ixz = "0">
-            </inertia>
-        </inertial>
-    </xacro:macro> -->
     <xacro:macro name = "wheel_link" params = "prefix">
         <link name = "${prefix}_wheel_link">
@@ -100,5 +87,5 @@
             <origin xyz = "0 0 ${base_height / 2.0}" rpy = "0 0 0" />
         </collision>
-        <xacro:box_inertia m = "${box_mass}" x="${base_length}" y="${base_width}" z="${base_height}" o_xyz="0 0 ${base_height / 2.0}" o_rpy="0 0 0" />
+        <xacro:box_inertia m = "${box_mass}" x = "${base_length}" y = "${base_width}" z = "${base_height}" o_xyz = "0 0 ${base_height / 2.0}" o_rpy = "0 0 0" />
     </link>
     <xacro:wheel_link prefix = "front_right" />
@@ -115,3 +102,6 @@
     <xacro:wheel_joint prefix = "back_right" x = "${-base_length / 4.0}" y = "${-(base_width + wheel_length) / 2.0}" />
     <xacro:wheel_joint prefix = "back_left" x = "${-base_length / 4.0}" y = "${(base_width + wheel_length) / 2.0}" />
+    <gazebo>
+        <plugin filename = "gz-sim-joint-state-publisher-system" name = "gz::sim::systems::JointStatePublisher" />
+    </gazebo>
 </robot>

Commit message: Add lidar_link

File: rover_description/urdf/rover.urdf.xacro (robot description, xacro)
@@ -102,4 +102,20 @@
     <xacro:wheel_joint prefix = "back_right" x = "${-base_length / 4.0}" y = "${-(base_width + wheel_length) / 2.0}" />
     <xacro:wheel_joint prefix = "back_left" x = "${-base_length / 4.0}" y = "${(base_width + wheel_length) / 2.0}" />
+    <link name = "lidar_link">
+        <visual>
+            <geometry>
+                <cylinder radius = "0.05" length = "0.02" />
+            </geometry>
+            <origin xyz = " 0 0 ${base_height}" rpy = "0 0 0" />
+            <material name = "green" />
+        </visual>
+        <collision>
+            <geometry>
+                <box size = "0.1 0.1 0.02" />
+            </geometry>
+            <origin xyz = " 0 0 ${base_height}" rpy = "0 0 0" />
+        </collision>
+        <xacro:box_inertia m = "0.2" x = "0.1" y = "0.1" z = "0.02" o_xyz = "0 0 ${base_height}" o_rpy = "0 0 0" />
+    </link>
     <gazebo>
         <plugin filename = "gz-sim-joint-state-publisher-system" name = "gz::sim::systems::JointStatePublisher" />

Commit message: Correcting origins

File: rover_description/urdf/rover.urdf.xacro (robot description, xacro)
@@ -107,5 +107,5 @@
                 <cylinder radius = "0.05" length = "0.02" />
             </geometry>
-            <origin xyz = " 0 0 ${base_height}" rpy = "0 0 0" />
+            <origin xyz = " 0 0 0" rpy = "0 0 0" />
             <material name = "green" />
         </visual>
@@ -114,7 +114,7 @@
                 <box size = "0.1 0.1 0.02" />
             </geometry>
-            <origin xyz = " 0 0 ${base_height}" rpy = "0 0 0" />
+            <origin xyz = " 0 0 0" rpy = "0 0 0" />
         </collision>
-        <xacro:box_inertia m = "0.2" x = "0.1" y = "0.1" z = "0.02" o_xyz = "0 0 ${base_height}" o_rpy = "0 0 0" />
+        <xacro:box_inertia m = "0.2" x = "0.1" y = "0.1" z = "0.02" o_xyz = "0 0 0" o_rpy = "0 0 0" />
     </link>
     <gazebo>

Commit message: Fix error

File: rover_description/urdf/rover.urdf.xacro (robot description, xacro)
@@ -107,5 +107,5 @@
                 <cylinder radius = "0.05" length = "0.02" />
             </geometry>
-            <origin xyz = " 0 0 0" rpy = "0 0 0" />
+            <origin xyz = "0 0 0" rpy = "0 0 0" />
             <material name = "green" />
         </visual>
@@ -114,5 +114,5 @@
                 <box size = "0.1 0.1 0.02" />
             </geometry>
-            <origin xyz = " 0 0 0" rpy = "0 0 0" />
+            <origin xyz = "0 0 0" rpy = "0 0 0" />
         </collision>
         <xacro:box_inertia m = "0.2" x = "0.1" y = "0.1" z = "0.02" o_xyz = "0 0 0" o_rpy = "0 0 0" />

Commit message: Add joint for lidar_link

File: rover_description/urdf/rover.urdf.xacro (robot description, xacro)
@@ -118,4 +118,9 @@
         <xacro:box_inertia m = "0.2" x = "0.1" y = "0.1" z = "0.02" o_xyz = "0 0 0" o_rpy = "0 0 0" />
     </link>
+    <joint>
+        <parent link = "base_link" />
+        <child link = "lidar_link" />
+        <origin xyz = "0 0 ${base_height / 2.0}" />
+    </joint>
     <gazebo>
         <plugin filename = "gz-sim-joint-state-publisher-system" name = "gz::sim::systems::JointStatePublisher" />

Commit message: Fix error of joint_name lidar_joint

File: rover_description/urdf/rover.urdf.xacro (robot description, xacro)
@@ -118,5 +118,5 @@
         <xacro:box_inertia m = "0.2" x = "0.1" y = "0.1" z = "0.02" o_xyz = "0 0 0" o_rpy = "0 0 0" />
     </link>
-    <joint>
+    <joint name = "lidar_joint">
         <parent link = "base_link" />
         <child link = "lidar_link" />

Commit message: Fix error of joint_type for lidar_joint

File: rover_description/urdf/rover.urdf.xacro (robot description, xacro)
@@ -118,5 +118,5 @@
         <xacro:box_inertia m = "0.2" x = "0.1" y = "0.1" z = "0.02" o_xyz = "0 0 0" o_rpy = "0 0 0" />
     </link>
-    <joint name = "lidar_joint">
+    <joint name = "lidar_joint" type = "fixed">
         <parent link = "base_link" />
         <child link = "lidar_link" />

Commit message: Fix origin of lidar_joint

File: rover_description/urdf/rover.urdf.xacro (robot description, xacro)
@@ -121,5 +121,5 @@
         <parent link = "base_link" />
         <child link = "lidar_link" />
-        <origin xyz = "0 0 ${base_height / 2.0}" />
+        <origin xyz = "0 0 ${base_height + 0.01}" />
     </joint>
     <gazebo>
