Commit message: Remove base_footprint

File: src/rover_description/urdf/rover.urdf.xacro (robot description, xacro)
@@ -74,5 +74,4 @@
     <xacro:property name = "box_mass" value = "5.0"/>
     <!-- TF Tree starts here -->
-    <link name = "base_footprint" />
     <link name = "base_link">
         <visual>
@@ -95,9 +94,4 @@
     <xacro:wheel_link prefix = "back_right" />
     <xacro:wheel_link prefix = "back_left" />
-    <joint name = "base_joint" type = "fixed">
-        <parent link = "base_footprint" />
-        <child link = "base_link" />
-        <origin xyz = "0 0 ${wheel_radius}" rpy = "0 0 0" />
-    </joint>
     <xacro:wheel_joint prefix = "front_right" x = "${base_length / 4.0}" y = "${-(base_width + wheel_length) / 2.0}" />
     <xacro:wheel_joint prefix = "front_left" x = "${base_length / 4.0}" y = "${(base_width + wheel_length) / 2.0}" />
@@ -171,5 +165,6 @@
             <use_pose_vector_msg>true</use_pose_vector_msg>
             <odom_frame>odom</odom_frame>
-            <base_frame>rover/base_footprint</base_frame>
+            <base_frame>base_link</base_frame>
+            <update_frequency>50</update_frequency>
         </plugin>
     </gazebo>
